Commit message: show stationary wheels in life setup

File: scout_description/urdf/scout_mini.xacro (robot description, xacro)
@@ -3,4 +3,5 @@
   <xacro:arg name="namespace" default=""/>
   <xacro:arg name="sim_reduction" default="2"/>
+  <xacro:arg name="sim" default="false"/>
   <xacro:include filename="$(find scout_description)/urdf/wheel.xacro"/>
   <!-- Variables -->
@@ -161,4 +162,6 @@
   </xacro:wheel>
   <!-- Gazebo sim definitions  -->
-  <xacro:include filename="$(find scout_description)/urdf/sim.gazebo"/>
+  <xacro:if value="${'$(arg sim)'}">
+    <xacro:include filename="$(find scout_description)/urdf/sim.gazebo"/>
+  </xacro:if>
 </robot>

File: scout_description/urdf/wheel.xacro (robot description, xacro)
@@ -45,31 +45,40 @@
       </collision>
     </link>
-    <joint name="${wheel_prefix}_wheel" type="continuous">
-      <parent link="base_link"/>
-      <child link="${wheel_prefix}_wheel_link"/>
-      <xacro:insert_block name="joint_pose"/>
-      <axis xyz="0 0 ${axis}" rpy="0 0 0"/>
-      <dynamics damping="0.0" friction="0.0"/>
-      <limit effort="1000" velocity="20"/>
-      <!-- High limits for fast turns -->
-    </joint>
-    <gazebo reference="${wheel_prefix}_wheel_link">
-      <!-- High for no longitudinal slip (propulsion) -->
-      <mu1>200.0</mu1>
-      <!-- High for lateral grip during turns (prevents sliding) -->
-      <mu2>0.7</mu2>
-      <!-- Small torsional slip for realism/stability -->
-      <slip1>0.01</slip1>
-      <!-- Lateral slip; tune higher (0.1) if turns feel too sticky -->
-      <slip2>0.01</slip2>
-      <!-- Stiffness: prevents sinking -->
-      <kp>1e7</kp>
-      <!-- Damping: reduces bounce; increased from 1.0 -->
-      <kd>10.0</kd>
-      <fdir1>1 0 0</fdir1>
-      <!-- Deeper contacts for better force transmission -->
-      <minDepth>0.005</minDepth>
-      <maxContacts>10</maxContacts>
-    </gazebo>
+    <xacro:if value="${'$(arg sim)'}">
+      <joint name="${wheel_prefix}_wheel" type="continuous">
+        <parent link="base_link"/>
+        <child link="${wheel_prefix}_wheel_link"/>
+        <xacro:insert_block name="joint_pose"/>
+        <axis xyz="0 0 ${axis}" rpy="0 0 0"/>
+        <dynamics damping="0.0" friction="0.0"/>
+        <limit effort="1000" velocity="20"/>
+        <!-- High limits for fast turns -->
+      </joint>
+      <gazebo reference="${wheel_prefix}_wheel_link">
+        <!-- High for no longitudinal slip (propulsion) -->
+        <mu1>200.0</mu1>
+        <!-- High for lateral grip during turns (prevents sliding) -->
+        <mu2>0.7</mu2>
+        <!-- Small torsional slip for realism/stability -->
+        <slip1>0.01</slip1>
+        <!-- Lateral slip; tune higher (0.1) if turns feel too sticky -->
+        <slip2>0.01</slip2>
+        <!-- Stiffness: prevents sinking -->
+        <kp>1e7</kp>
+        <!-- Damping: reduces bounce; increased from 1.0 -->
+        <kd>10.0</kd>
+        <fdir1>1 0 0</fdir1>
+        <!-- Deeper contacts for better force transmission -->
+        <minDepth>0.005</minDepth>
+        <maxContacts>10</maxContacts>
+      </gazebo>
+    </xacro:if>
+    <xacro:unless value="${'$(arg sim)'}">
+      <joint name="${wheel_prefix}_wheel" type="fixed">
+        <parent link="base_link"/>
+        <child link="${wheel_prefix}_wheel_link"/>
+        <xacro:insert_block name="joint_pose"/>
+      </joint>
+    </xacro:unless>
   </xacro:macro>
 </robot>

Commit message: use real realsense camera description in xacro

File: scout_description/urdf/scout_mini.xacro (robot description, xacro)
@@ -5,4 +5,5 @@
   <xacro:arg name="sim" default="false"/>
   <xacro:include filename="$(find scout_description)/urdf/wheel.xacro"/>
+  <xacro:include filename="$(find realsense2_description)/urdf/_d435.urdf.xacro" />
   <!-- Variables -->
   <xacro:property name="M_PI" value="3.14159"/>
@@ -33,6 +34,4 @@
       <origin xyz="0 0 0" rpy="0 0 0"/>
       <geometry>
-        <!-- <mesh
-              filename="package://scout_description/meshes/scout_mini_base_link2.dae" /> -->
         <box size="0.4 0.4 0.05"/>
       </geometry>
@@ -41,5 +40,5 @@
   <link name="box_link">
     <inertial>
-      <origin xyz="0.0 0.0 0.0" rpy="0 0 3.14159"/>
+      <origin xyz="0.0 0.0 0.0" rpy="0 0 ${M_PI}"/>
       <mass value="5"/>
       <inertia ixx="0.054166666667" ixy="0" ixz="0" iyy="0.075" iyz="0" izz="0.054166666667"/>
@@ -88,26 +87,5 @@
     <child link="laser_link"/>
   </joint>
-  <link name="camera_link">
-    <inertial>
-      <origin xyz="0.0 0.0 0.0" rpy="0 0 0"/>
-      <mass value="0.1"/>
-      <inertia ixx="0.0088463" ixy="2.0356E-05" ixz="-0.00047464" iyy="0.0066478" iyz="-6.9288E-06" izz="0.01219"/>
-    </inertial>
-    <visual>
-      <origin xyz="0.0 0.0 0.0" rpy="0.0 0.0 0.0"/>
-      <geometry>
-        <mesh filename="package://scout_description/meshes/box-parts/camera.stl"/>
-      </geometry>
-      <material name="red">
-        <color rgba="1 0 0 1"/>
-      </material>
-    </visual>
-    <collision>
-      <origin xyz="0 0 0.31" rpy="0 0 0"/>
-      <geometry>
-        <box size="0.01 0.01 0.01"/>
-      </geometry>
-    </collision>
-  </link>
+  <link name="camera_link"/>
   <joint name="camera_joint" type="fixed">
     <origin xyz="0.192646 -0.001255 0.096" rpy="0 0 0"/>
@@ -115,10 +93,10 @@
     <child link="camera_link"/>
   </joint>
-  <link name="camera_optical_link"/>
-  <joint name="camera_optical_joint" type="fixed">
-    <origin xyz="0.01495 0 0.0125" rpy="0 0 0"/>
-    <parent link="camera_link"/>
-    <child link="camera_optical_link"/>
-  </joint>
+  <xacro:sensor_d435
+    name="d435_camera"
+    parent="camera_link"
+    use_nominal_extrinsics="$(arg sim)">
+    <origin xyz="0 0 0" rpy="0 0 0" />
+  </xacro:sensor_d435>
   <link name="monitor_link">
     <inertial>

Commit message: add dummy imu_link

File: scout_description/urdf/scout_mini.xacro (robot description, xacro)
@@ -64,4 +64,10 @@
     <parent link="base_link"/>
     <child link="box_link"/>
+  </joint>
+  <link name="imu_link"/>
+  <joint name="imu_joint" type="fixed">
+    <origin xyz="0 0 0" rpy="0 0 0"/>
+    <parent link="box_link"/>
+    <child link="imu_link"/>
   </joint>
   <link name="laser_link">

Commit message: remove unnecessary wheel radius from definition

File: scout_description/urdf/scout_mini.xacro (robot description, xacro)
@@ -18,5 +18,4 @@
   <xacro:property name="wheel_width" value="0.084"/>
   <xacro:property name="wheel_length" value="0.8e-01"/>
-  <xacro:property name="wheel_radius" value="1.600e-01"/>
   <link name="base_link">
     <inertial>
